Commit message: .

File: src/obs_avoidance/urdf/rover.xacro (robot description, xacro)
@@ -1,26 +1,6 @@
 <?xml version='1.0'?>
-<robot name="rover" xmlns:xacro="http://www.ros.org/wiki/xacro">
-<xacro:include filename="$(find obs_avoidance)/urdf/rover.gazebo" />
-<!-- CAMERAS-->
-<link name="hokuyo">
-    <collision>
-      <origin xyz="0 0 0" rpy="0 0 0"/>
-      <geometry>
-         <box size="0.1 0.1 0.1"/>
-      </geometry>
-    </collision>
-    <visual>
-      <origin xyz="0 0 0" rpy="0 0 0"/>
-      <geometry>
-        <mesh filename="package://gazebo_bot/meshes/hokuyo.dae"/>
-      </geometry>
-    </visual>
-    <inertial>
-      <mass value="1e-5" />
-      <origin xyz="0 0 0" rpy="0 0 0"/>
-      <inertia ixx="1e-6" ixy="0" ixz="0" iyy="1e-6" iyz="0" izz="1e-6" />
-    </inertial>
-</link>
-<!-- CHASSIS -->
+<robot name="mybot" xmlns:xacro="http://www.ros.org/wiki/xacro">
+<xacro:include filename="$(find mybot_description)/urdf/rover.gazebo" />
+<xacro:include filename="$(find realsense2_description)/urdf/_d435.urdf.xacro"/>
   <link name="chassis">
     <pose>0 0 0.1 0 0 0</pose>
@@ -36,5 +16,5 @@
     <collision name='collision'>
       <geometry>
-        <box size="1 1 .1"/>
+        <box size="1.0 1.0 .1"/>
       </geometry>
     </collision>
@@ -42,11 +22,49 @@
       <origin xyz="0 0 0" rpy=" 0 0 0"/>
       <geometry>
-        <box size="1 1 .1"/>
-      </geometry>
-    </visual>
-  </link>
-<!-- WHEEL LINKS -->
+        <box size="1.0 1.0 .1"/>
+      </geometry>
+    </visual>
+  </link>
+<!--link name="camera">
+        <collision name="collision_camera">
+                <origin xyz="0 0 0" rpy="0 0 0" />
+                <geometry>
+                         <box size="0.1 0.1 0.1" />
+                </geometry>
+        </collision>
+        <visual name="camera_visual">
+                <origin xyz="0 0 0" rpy="0 0 0" />
+                <geometry>
+                        <box size="0.1 0.1 0.1" />
+                </geometry>
+        </visual>
+        <inertial>
+                <mass value="0.1" />
+                <origin xyz="0 0 0.0001" rpy="0 0 0"/>
+                <inertia ixx="0.0001" ixy="0.0" ixz="0.0"
+                         iyy="0.0001" iyz="0.0"
+                         izz="0.0001" />
+        </inertial>
+</link-->
+<link name="hokuyo">
+    <collision>
+      <origin xyz="0 0 0" rpy="0 0 0"/>
+      <geometry>
+         <box size="0.1 0.1 0.1"/>
+      </geometry>
+    </collision>
+    <visual>
+      <origin xyz="0 0 0" rpy="0 0 0"/>
+      <geometry>
+        <mesh filename="package://mybot_description/meshes/hokuyo.dae"/>
+      </geometry>
+    </visual>
+    <inertial>
+      <mass value="1e-5" />
+      <origin xyz="0 0 0" rpy="0 0 0"/>
+      <inertia ixx="1e-6" ixy="0" ixz="0" iyy="1e-6" iyz="0" izz="1e-6" />
+    </inertial>
+</link>
   <link name="left_wheel">
-    <!--origin xyz="0.1 0.13 0.1" rpy="0 1.5707 1.5707"-->
     <collision name="collision">
       <origin xyz="0 0 0" rpy="0 1.5707 1.5707"/>
@@ -72,5 +90,4 @@
   </link>
   <link name="right_wheel">
-    <!--origin xyz="0.1 -0.13 0.1" rpy="0 1.5707 1.5707"/-->
     <collision name="collision">
       <origin xyz="0 0 0" rpy="0 1.5707 1.5707"/>
@@ -96,5 +113,4 @@
   </link>
   <link name="left_fwheel">
-    <!--origin xyz="-0.1 0.13 0.1" rpy="0 1.5707 1.5707"-->
     <collision name="collision">
       <origin xyz="0 0 0" rpy="0 1.5707 1.5707"/>
@@ -120,5 +136,4 @@
   </link>
   <link name="right_fwheel">
-    <!--origin xyz="-0.1 -0.13 0.1" rpy="0 1.5707 1.5707"/-->
     <collision name="collision">
       <origin xyz="0 0 0" rpy="0 1.5707 1.5707"/>
@@ -143,42 +158,43 @@
     </inertial>
   </link>
-<!--JOINTS -->
+  <joint type="continuous" name="left_wheel_hinge">
+    <origin xyz="0.25 0.565 0" rpy="0 0 0"/>
+    <child link="left_wheel"/>
+    <parent link="chassis"/>
+    <axis xyz="0 1 0" rpy="0 0 0"/>
+    <limit effort="100" velocity="100"/>
+    <joint_properties damping="0.0" friction="1.0"/>
+  </joint>
+  <joint type="continuous" name="right_wheel_hinge">
+    <origin xyz="0.25 -0.565 0" rpy="0 0 0"/>
+    <child link="right_wheel"/>
+    <parent link="chassis"/>
+    <axis xyz="0 1 0" rpy="0 0 0"/>
+    <limit effort="100" velocity="100"/>
+    <joint_properties damping="0.0" friction="1.0"/>
+  </joint>
+ <joint type="continuous" name="left_wheel_fhinge">
+    <origin xyz="-0.25 0.565 0" rpy="0 0 0"/>
+    <child link="left_fwheel"/>
+    <parent link="chassis"/>
+    <axis xyz="0 1 0" rpy="0 0 0"/>
+    <limit effort="100" velocity="100"/>
+    <joint_properties damping="0.0" friction="1.0"/>
+  </joint>
+  <joint type="continuous" name="right_wheel_fhinge">
+    <origin xyz="-0.25 -0.565 0" rpy="0 0 0"/>
+    <child link="right_fwheel"/>
+    <parent link="chassis"/>
+    <axis xyz="0 1 0" rpy="0 0 0"/>
+    <limit effort="100" velocity="100"/>
+    <joint_properties damping="0.0" friction="1"/>
+  </joint>
 <joint name="hokuyo_joint" type="fixed">
-        <origin xyz="-0.45 0 0.25" rpy="0 0 3.1414" />
+        <origin xyz="0.45 0 0.25" rpy="0 0 0" />
         <child link="hokuyo" />
         <parent link="chassis" />
 </joint>
-  <joint type="continuous" name="left_wheel_hinge">
-    <origin xyz="0.25 0.565 0" rpy="0 0 0"/>
-    <child link="left_wheel"/>
-    <parent link="chassis"/>
-    <axis xyz="0 1 0" rpy="0 0 0"/>
-    <limit effort="100" velocity="100"/>
-    <joint_properties damping="0.0" friction="1.0"/>
-  </joint>
-  <joint type="continuous" name="right_wheel_hinge">
-    <origin xyz="0.25 -0.565 0" rpy="0 0 0"/>
-    <child link="right_wheel"/>
-    <parent link="chassis"/>
-    <axis xyz="0 1 0" rpy="0 0 0"/>
-    <limit effort="100" velocity="100"/>
-    <joint_properties damping="0.0" friction="1.0"/>
-  </joint>
- <joint type="continuous" name="left_wheel_fhinge">
-    <origin xyz="-0.25 0.565 0" rpy="0 0 0"/>
-    <child link="left_fwheel"/>
-    <parent link="chassis"/>
-    <axis xyz="0 1 0" rpy="0 0 0"/>
-    <limit effort="100" velocity="100"/>
-    <joint_properties damping="0.0" friction="1.0"/>
-  </joint>
-  <joint type="continuous" name="right_wheel_fhinge">
-    <origin xyz="-0.25 -0.565 0" rpy="0 0 0"/>
-    <child link="right_fwheel"/>
-    <parent link="chassis"/>
-    <axis xyz="0 1 0" rpy="0 0 0"/>
-    <limit effort="100" velocity="100"/>
-    <joint_properties damping="0.0" friction="1"/>
-  </joint>
-<!-- END -->
+<sensor_d435 parent="chassis" name="camera" >
+        <origin xyz="0.45 0 0.3" rpy="0 0 0" />
+</sensor_d435>
 </robot>
